File: lipo-charger/lipo-charger.kicad_pcb (KiCad board)
At the start: 2 copper layers, 39.4 x 25.4 mm, 14 parts, among them J1 USB_B_Micro, U1 MCP73831-2-OT

Commit message: add connector
Parts:
- added J2: Screw_Terminal_01x02, Connector_Molex:Molex_KK-254_AE-6410-02A_1x02_P2.54mm_Vertical, F.Cu at (121.9, 61.0)
- added J3: Conn_01x02, Connector_JST:JST_PH_B2B-PH-K_1x02_P2.00mm_Vertical, F.Cu at (122.0, 67.6)
- added TP1: TestPoint, Connector_Pin:Pin_D0.7mm_L6.5mm_W1.8mm_FlatFork, F.Cu at (114.3, 52.5)
- added TP2: TestPoint, Connector_Pin:Pin_D0.7mm_L6.5mm_W1.8mm_FlatFork, F.Cu at (111.4, 52.5)
- renumbered CHARGING to D1, 50ma to JP1, 100ma to JP2, 250ma to JP3, 500ma to JP4

Commit message: update test + final wiring
Parts:
- renumbered JP2 to 100ma, JP3 to 200ma, JP4 to 500ma, JP1 to 50ma
Connections:
- J2 pad 1: unconnected-(J2-Pin_1-Pad1) -> LIPO
- J2 pad 2: unconnected-(J2-Pin_2-Pad2) -> GND
- J3 pad 1: unconnected-(J3-Pin_1-Pad1) -> LIPO
- J3 pad 2: unconnected-(J3-Pin_2-Pad2) -> GND
- TP1 pad 1: unconnected-(TP1-Pad1) -> LIPO
- TP2 pad 1: unconnected-(TP2-Pad1) -> GND
Routing:
- net LIPO: track 0.00 -> 38.4 mm
- net PROG: track 0.00 -> 20.5 mm
- net +5V: track 0.00 -> 19.7 mm
- net Net-(U1-STAT): track 0.00 -> 14.5 mm, vias 0 -> 2
- net Net-(D1-K): track 0.00 -> 3.54 mm
- net Net-(JP4-A): track 0.00 -> 3.11 mm
- net Net-(JP3-A): track 0.00 -> 3.09 mm
- net Net-(JP2-A): track 0.00 -> 3.06 mm
- net Net-(JP1-A): track 0.00 -> 3.03 mm
- net GND: track 0.00 -> 2.22 mm, vias 0 -> 6
- added copper zone on B.Cu, net GND
- added copper zone on F.Cu, net GND
